File: Hardware/Qwiic Shield for RaspberryPi.sch (EAGLE design)
At the start: 19 parts, among them U2 3.3V/600mA, U3 RASPBERRY_PI

Commit message: Adding panel files
Parts:
- U$2: value SPARKX-LOGO5 -> SPARKX-LOGO4; device SparkX:SPARKX-LOGO5 -> SparkX:SPARKX-LOGO4
- U3: device SparkX:RASPBERRY_PI_40SMD -> SparkX:RASPBERRY_PI_40BTM-NOHOLES
Connections:
- net D13: no longer J4.4
- net D16: now also J4.4
- net D19: no longer J4.5
- net D20: now also J4.5
- net D21: now also J4.6
- net D26: no longer J4.6
- net D5: no longer J4.1
- net D7: now also J4.1
- net SCL: now also J12.2; no longer J12.1
- net SDA: now also J12.1; no longer J12.2
Other:
- note removed: "Add keep out ring to drill hits"
- note removed: "Create addtional fps without drills"
- note removed: "How much can ESP and Photon provide over 3.3V? Remove 3.3V reg?"
Changed lines of the file:
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@@
 <?xml version="1.0" encoding="utf-8"?>
 <!DOCTYPE eagle SYSTEM "eagle.dtd">
-<eagle version="7.5.0">
+<eagle version="7.7.0">
 <drawing>
 <settings>
@@
 <layer number="230" name="230bmp" color="7" fill="1" visible="yes" active="yes"/>
 <layer number="231" name="231bmp" color="7" fill="1" visible="yes" active="yes"/>
+<layer number="232" name="Eagle3D_PG2" color="7" fill="1" visible="yes" active="yes"/>
+<layer number="233" name="Eagle3D_PG3" color="7" fill="1" visible="yes" active="yes"/>
 <layer number="248" name="Housing" color="7" fill="1" visible="yes" active="yes"/>
 <layer number="249" name="Edge" color="7" fill="1" visible="yes" active="yes"/>
@@
 <part name="J4" library="SparkFun-Connectors" deviceset="CONN_06" device="NO_SILK_FEMALE_PTH"/>
 <part name="U$1" library="SparkX" deviceset="SPARKX-LOGO" device="3"/>
-<part name="U$2" library="SparkX" deviceset="SPARKX-LOGO" device="5" value="SPARKX-LOGO5"/>
-<part name="U3" library="SparkX" deviceset="RASPBERRY_PI_40" device="SMD" value="RASPBERRY_PI"/>
+<part name="U$2" library="SparkX" deviceset="SPARKX-LOGO" device="4" value="SPARKX-LOGO4"/>
+<part name="U3" library="SparkX" deviceset="RASPBERRY_PI_40" device="BTM-NOHOLES" value="RASPBERRY_PI"/>
 <part name="SUPPLY11" library="SparkFun-PowerSymbols" deviceset="5V" device=""/>
 <part name="GND21" library="SparkFun" deviceset="GND" device=""/>
@@
 <text x="111.76" y="157.48" size="3.048" layer="97" font="vector" ratio="12" align="center">Proto Connections</text>
 <text x="157.48" y="134.62" size="3.048" layer="97" font="vector" ratio="12" align="center">Power</text>
-<text x="152.4" y="55.88" size="1.27" layer="91" align="center">How much can ESP and Photon provide over 3.3V? Remove 3.3V reg?</text>
-<text x="149.86" y="58.42" size="1.27" layer="91" align="center">Create addtional fps without drills</text>
-<text x="149.86" y="60.96" size="1.27" layer="91" align="center">Add keep out ring to drill hits</text>
 </plain>
 <instances>
@@
 <segment>
 <pinref part="U3" gate="U1" pin="SDA/D2"/>
-<wire x1="66.04" y1="134.62" x2="83.82" y2="134.62" width="0.1524" layer="91"/>
-<label x="83.82" y="134.62" size="1.27" layer="95" xref="yes"/>
+<wire x1="66.04" y1="134.62" x2="71.12" y2="134.62" width="0.1524" layer="91"/>
+<label x="71.12" y="134.62" size="1.27" layer="95" xref="yes"/>
 </segment>
 <segment>
@@
 </segment>
 <segment>
+<pinref part="J12" gate="G$1" pin="1"/>
+<wire x1="109.22" y1="114.3" x2="106.68" y2="114.3" width="0.1524" layer="91"/>
+<label x="106.68" y="114.3" size="1.27" layer="95" rot="R180" xref="yes"/>
+</segment>
+</net>
+<net name="SCL" class="0">
+<segment>
+<pinref part="U3" gate="U1" pin="SCL/D3"/>
+<wire x1="66.04" y1="132.08" x2="71.12" y2="132.08" width="0.1524" layer="91"/>
+<label x="71.12" y="132.08" size="1.27" layer="95" xref="yes"/>
+</segment>
+<segment>
+<pinref part="J1" gate="G$1" pin="SCL"/>
+<wire x1="213.36" y1="144.78" x2="218.44" y2="144.78" width="0.1524" layer="91"/>
+<label x="218.44" y="144.78" size="1.27" layer="95" xref="yes"/>
+</segment>
+<segment>
+<pinref part="J6" gate="G$1" pin="SCL"/>
+<wire x1="213.36" y1="121.92" x2="218.44" y2="121.92" width="0.1524" layer="91"/>
+<label x="218.44" y="121.92" size="1.27" layer="95" xref="yes"/>
+</segment>
+<segment>
+<pinref part="J7" gate="G$1" pin="SCL"/>
+<wire x1="213.36" y1="96.52" x2="218.44" y2="96.52" width="0.1524" layer="91"/>
+<label x="218.44" y="96.52" size="1.27" layer="95" xref="yes"/>
+</segment>
+<segment>
+<pinref part="J8" gate="G$1" pin="SCL"/>
+<wire x1="213.36" y1="68.58" x2="218.44" y2="68.58" width="0.1524" layer="91"/>
+<label x="218.44" y="68.58" size="1.27" layer="95" xref="yes"/>
+</segment>
+<segment>
 <pinref part="J12" gate="G$1" pin="2"/>
 <wire x1="109.22" y1="111.76" x2="106.68" y2="111.76" width="0.1524" layer="91"/>
 <label x="106.68" y="111.76" size="1.27" layer="95" rot="R180" xref="yes"/>
-</segment>
-</net>
-<net name="SCL" class="0">
-<segment>
-<pinref part="U3" gate="U1" pin="SCL/D3"/>
-<wire x1="66.04" y1="132.08" x2="83.82" y2="132.08" width="0.1524" layer="91"/>
-<label x="83.82" y="132.08" size="1.27" layer="95" xref="yes"/>
-</segment>
-<segment>
-<pinref part="J1" gate="G$1" pin="SCL"/>
-<wire x1="213.36" y1="144.78" x2="218.44" y2="144.78" width="0.1524" layer="91"/>
-<label x="218.44" y="144.78" size="1.27" layer="95" xref="yes"/>
-</segment>
-<segment>
-<pinref part="J6" gate="G$1" pin="SCL"/>
-<wire x1="213.36" y1="121.92" x2="218.44" y2="121.92" width="0.1524" layer="91"/>
-<label x="218.44" y="121.92" size="1.27" layer="95" xref="yes"/>
-</segment>
-<segment>
-<pinref part="J7" gate="G$1" pin="SCL"/>
-<wire x1="213.36" y1="96.52" x2="218.44" y2="96.52" width="0.1524" layer="91"/>
-<label x="218.44" y="96.52" size="1.27" layer="95" xref="yes"/>
-</segment>
-<segment>
-<pinref part="J8" gate="G$1" pin="SCL"/>
-<wire x1="213.36" y1="68.58" x2="218.44" y2="68.58" width="0.1524" layer="91"/>
-<label x="218.44" y="68.58" size="1.27" layer="95" xref="yes"/>
-</segment>
-<segment>
-<pinref part="J12" gate="G$1" pin="1"/>
-<wire x1="109.22" y1="114.3" x2="106.68" y2="114.3" width="0.1524" layer="91"/>
-<label x="106.68" y="114.3" size="1.27" layer="95" rot="R180" xref="yes"/>
 </segment>
 </net>
@@
 <label x="71.12" y="111.76" size="1.27" layer="95" xref="yes"/>
 </segment>
+</net>
+<net name="D6" class="0">
+<segment>
+<pinref part="U3" gate="U1" pin="D6"/>
+<wire x1="71.12" y1="109.22" x2="66.04" y2="109.22" width="0.1524" layer="91"/>
+<label x="71.12" y="109.22" size="1.27" layer="95" xref="yes"/>
+</segment>
+<segment>
+<pinref part="J4" gate="G$1" pin="3"/>
+<wire x1="109.22" y1="78.74" x2="106.68" y2="78.74" width="0.1524" layer="91"/>
+<label x="106.68" y="78.74" size="1.27" layer="95" rot="R180" xref="yes"/>
+</segment>
+</net>
+<net name="D7" class="0">
+<segment>
+<pinref part="U3" gate="U1" pin="D7"/>
+<wire x1="71.12" y1="106.68" x2="66.04" y2="106.68" width="0.1524" layer="91"/>
+<label x="71.12" y="106.68" size="1.27" layer="95" xref="yes"/>
+</segment>
 <segment>
 <pinref part="J4" gate="G$1" pin="1"/>
@@
 </segment>
 </net>
-<net name="D6" class="0">
-<segment>
-<pinref part="U3" gate="U1" pin="D6"/>
-<wire x1="71.12" y1="109.22" x2="66.04" y2="109.22" width="0.1524" layer="91"/>
-<label x="71.12" y="109.22" size="1.27" layer="95" xref="yes"/>
-</segment>
-<segment>
-<pinref part="J4" gate="G$1" pin="3"/>
-<wire x1="109.22" y1="78.74" x2="106.68" y2="78.74" width="0.1524" layer="91"/>
-<label x="106.68" y="78.74" size="1.27" layer="95" rot="R180" xref="yes"/>
-</segment>
-</net>
-<net name="D7" class="0">
-<segment>
-<pinref part="U3" gate="U1" pin="D7"/>
-<wire x1="71.12" y1="106.68" x2="66.04" y2="106.68" width="0.1524" layer="91"/>
-<label x="71.12" y="106.68" size="1.27" layer="95" xref="yes"/>
-</segment>
-</net>
 <net name="D12" class="0">
 <segment>
@@
 <label x="71.12" y="101.6" size="1.27" layer="95" xref="yes"/>
 </segment>
+</net>
+<net name="D16" class="0">
+<segment>
+<pinref part="U3" gate="U1" pin="D16"/>
+<wire x1="71.12" y1="99.06" x2="66.04" y2="99.06" width="0.1524" layer="91"/>
+<label x="71.12" y="99.06" size="1.27" layer="95" xref="yes"/>
+</segment>
 <segment>
 <pinref part="J4" gate="G$1" pin="4"/>
@@
 </segment>
 </net>
-<net name="D16" class="0">
-<segment>
-<pinref part="U3" gate="U1" pin="D16"/>
-<wire x1="71.12" y1="99.06" x2="66.04" y2="99.06" width="0.1524" layer="91"/>
-<label x="71.12" y="99.06" size="1.27" layer="95" xref="yes"/>
-</segment>
-</net>
 <net name="D17" class="0">
 <segment>
@@
 <label x="71.12" y="91.44" size="1.27" layer="95" xref="yes"/>
 </segment>
+</net>
+<net name="D20" class="0">
+<segment>
+<pinref part="U3" gate="U1" pin="D20"/>
+<wire x1="71.12" y1="88.9" x2="66.04" y2="88.9" width="0.1524" layer="91"/>
+<label x="71.12" y="88.9" size="1.27" layer="95" xref="yes"/>
+</segment>
 <segment>
 <pinref part="J4" gate="G$1" pin="5"/>
@@
 </segment>
 </net>
-<net name="D20" class="0">
-<segment>
-<pinref part="U3" gate="U1" pin="D20"/>
-<wire x1="71.12" y1="88.9" x2="66.04" y2="88.9" width="0.1524" layer="91"/>
-<label x="71.12" y="88.9" size="1.27" layer="95" xref="yes"/>
-</segment>
-</net>
 <net name="D21" class="0">
 <segment>
@@
 <label x="71.12" y="86.36" size="1.27" layer="95" xref="yes"/>
 </segment>
+<segment>
+<pinref part="J4" gate="G$1" pin="6"/>
+<wire x1="109.22" y1="71.12" x2="106.68" y2="71.12" width="0.1524" layer="91"/>
+<label x="106.68" y="71.12" size="1.27" layer="95" rot="R180" xref="yes"/>
+</segment>
 </net>
 <net name="D22" class="0">
@@
 <label x="71.12" y="73.66" size="1.27" layer="95" xref="yes"/>
 </segment>
-<segment>
-<pinref part="J4" gate="G$1" pin="6"/>
-<wire x1="109.22" y1="71.12" x2="106.68" y2="71.12" width="0.1524" layer="91"/>
-<label x="106.68" y="71.12" size="1.27" layer="95" rot="R180" xref="yes"/>
-</segment>
-</net>
+</net>
