File: Hardware/Panel/Qwiic_Shield_RaspberryPi-Panel.brd (EAGLE design)
At the start: 52.3 x 23 mm, 19 parts, among them U2 3.3V/600mA, U3 RASPBERRY_PI

Commit message: Adding panel files
Parts:
- removed FRAME1: FRAME-LETTER, SparkFun-Aesthetics:CREATIVE_COMMONS
- added C10, C11, C12, C13, C14, C15, C16, C2, C4, C5, C6, C7, C8, C9: 1.0uF, SparkFun-Capacitors:0603
- added FD10, FD11, FD12, FD13, FD14, FD15, FD16, FD3, FD4, FD5, FD6, FD7, FD8, FD9: FIDUCIAL1X2, SparkFun-Aesthetics:FIDUCIAL-1X2
- added J10, J20, J29, J38, J47, J56, J65: (no value), SparkFun-Connectors:1X06_NO_SILK
- added J11, J13, J21, J22, J30, J31, J39, J40, J48, J49, J57, J58, J66, J67: (no value), SparkFun-Connectors:1X02_NO_SILK
- added J14, J15, J23, J24, J32, J33, J41, J42, J50, J51, J59, J60, J68, J69: (no value), SparkFun-Connectors:1X04_NO_SILK
- added J16, J17, J18, J19, J25, J26, J27, J28, J34, J35, J36, J37, J43, J44, J45, J46, J52, J53, J54, J55, J61, J62, J63, J64, J70, J71, J72, J9: (no value), SparkX:1X04_1MM_RA
- added LOGO2, LOGO3, LOGO4, LOGO5, LOGO6, LOGO7, LOGO8: OSHW-LOGOMINI, SparkFun-Aesthetics:OSHW-LOGO-MINI
- added U$10, U$12, U$14, U$16, U$4, U$6, U$8: SPARKX-LOGO4, SparkX:SPARKX-MEDIUM
- added U$11, U$13, U$15, U$3, U$5, U$7, U$9: SPARKX-LOGO3, SparkX:SPARKX-SMALL
- added U1, U11, U13, U15, U5, U7, U9: RASPBERRY_PI, SparkX:RASPBERRY_PI_SHIELD_BOTTOM_ENTRY_NOHOLES
- added U10, U12, U14, U16, U4, U6, U8: 3.3V/600mA, SparkFun-IC-Power:SOT23-5
Connections:
- new net 3.3V1: C4.1, J15.2, J16.2, J17.2, J18.2, J9.2, U4.5
- new net 3.3V2: C6.1, J19.2, J24.2, J25.2, J26.2, J27.2, U6.5
- new net 3.3V3: C8.1, J28.2, J33.2, J34.2, J35.2, J36.2, U8.5
- new net 3.3V4: C10.1, J37.2, J42.2, J43.2, J44.2, J45.2, U10.5
- new net 3.3V5: C12.1, J46.2, J51.2, J52.2, J53.2, J54.2, U12.5
- new net 3.3V6: C14.1, J55.2, J60.2, J61.2, J62.2, J63.2, U14.5
- new net 3.3V7: C16.1, J64.2, J69.2, J70.2, J71.2, J72.2, U16.5
- new net 5V1: C2.1, J15.1, U1.2, U1.4, U4.1, U4.3
- new net 5V2: C5.1, J24.1, U5.2, U5.4, U6.1, U6.3
- new net 5V3: C7.1, J33.1, U7.2, U7.4, U8.1, U8.3
- new net 5V4: C9.1, J42.1, U10.1, U10.3, U9.2, U9.4
- new net 5V5: C11.1, J51.1, U11.2, U11.4, U12.1, U12.3
- new net 5V6: C13.1, J60.1, U13.2, U13.4, U14.1, U14.3
- new net 5V7: C15.1, J69.1, U15.2, U15.4, U16.1, U16.3
- new net CS1: J14.4, U1.24
- new net CS2: J23.4, U5.24
- new net CS3: J32.4, U7.24
- new net CS4: J41.4, U9.24
- new net CS5: J50.4, U11.24
- new net CS6: J59.4, U13.24
- new net CS7: J68.4, U15.24
- new net D1: U1.29
- new net D10: J10.4, U1.36
- new net D100: J47.5, U11.38
- new net D101: J47.6, U11.40
- new net D102: U11.15
- new net D103: U11.16
- new net D104: U11.18
- new net D105: U11.22
- new net D106: U11.37
- new net D107: U11.13
- new net D108: U11.7
- new net D109: U13.29
- new net D11: U1.11
- new net D110: J56.3, U13.31
- new net D111: J56.1, U13.26
- new net D112: J56.2, U13.32
- new net D113: U13.33
- new net D114: J56.4, U13.36
- new net D115: U13.11
- new net D116: U13.12
- new net D117: U13.35
- new net D118: J56.5, U13.38
- new net D119: J56.6, U13.40
- new net D120: U13.15
- new net D121: U13.16
- new net D122: U13.18
- new net D123: U13.22
- new net D124: U13.37
- new net D125: U13.13
- new net D126: U13.7
- new net D127: U15.29
- new net D128: J65.3, U15.31
- new net D129: J65.1, U15.26
- new net D130: J65.2, U15.32
- new net D131: U15.33
- new net D132: J65.4, U15.36
- new net D133: U15.11
- new net D134: U15.12
- new net D135: U15.35
- new net D136: J65.5, U15.38
- new net D137: J65.6, U15.40
- new net D138: U15.15
- new net D139: U15.16
- new net D14: U1.12
- new net D140: U15.18
- new net D141: U15.22
- new net D142: U15.37
- new net D143: U15.13
- new net D144: U15.7
- new net D15: U1.35
- new net D2: J10.3, U1.31
- new net D28: J10.5, U1.38
- new net D29: J10.6, U1.40
- new net D3: J10.1, U1.26
- new net D30: U1.15
- new net D31: U1.16
- new net D32: U1.18
- new net D33: U1.22
- new net D34: U1.37
- new net D35: U1.13
- new net D36: U1.7
- new net D37: U5.29
- new net D38: J20.3, U5.31
- new net D39: J20.1, U5.26
- new net D40: J20.2, U5.32
- new net D41: U5.33
- new net D42: J20.4, U5.36
- new net D43: U5.11
- new net D44: U5.12
- new net D45: U5.35
- new net D46: J20.5, U5.38
- new net D47: J20.6, U5.40
- new net D48: U5.15
- new net D49: U5.16
- new net D50: U5.18
- new net D51: U5.22
- new net D52: U5.37
- new net D53: U5.13
- new net D54: U5.7
- new net D55: U7.29
- new net D56: J29.3, U7.31
- new net D57: J29.1, U7.26
- new net D58: J29.2, U7.32
- new net D59: U7.33
- new net D60: J29.4, U7.36
- new net D61: U7.11
- new net D62: U7.12
- new net D63: U7.35
- new net D64: J29.5, U7.38
- new net D65: J29.6, U7.40
- new net D66: U7.15
- new net D67: U7.16
- new net D68: U7.18
- new net D69: U7.22
- new net D70: U7.37
- new net D71: U7.13
- new net D72: U7.7
- new net D73: U9.29
- new net D74: J38.3, U9.31
- new net D75: J38.1, U9.26
- new net D76: J38.2, U9.32
- new net D77: U9.33
- new net D78: J38.4, U9.36
- new net D79: U9.11
- new net D8: J10.2, U1.32
- new net D80: U9.12
- new net D81: U9.35
- new net D82: J38.5, U9.38
- new net D83: J38.6, U9.40
- new net D84: U9.15
- new net D85: U9.16
- new net D86: U9.18
- new net D87: U9.22
- new net D88: U9.37
- new net D89: U9.13
- new net D9: U1.33
- new net D90: U9.7
- new net D91: U11.29
- new net D92: J47.3, U11.31
- new net D93: J47.1, U11.26
- new net D94: J47.2, U11.32
- new net D95: U11.33
- new net D96: J47.4, U11.36
- new net D97: U11.11
- new net D98: U11.12
- new net D99: U11.35
- new net GND1: C2.2, C4.2, J15.3, J15.4, J16.1, J17.1, J18.1, J9.1, U1.14, U1.20, U1.25, U1.30, U1.34, U1.39, U1.6, U1.9, U4.2
- new net GND2: C5.2, C6.2, J19.1, J24.3, J24.4, J25.1, J26.1, J27.1, U5.14, U5.20, U5.25, U5.30, U5.34, U5.39, U5.6, U5.9, U6.2
- new net GND3: C7.2, C8.2, J28.1, J33.3, J33.4, J34.1, J35.1, J36.1, U7.14, U7.20, U7.25, U7.30, U7.34, U7.39, U7.6, U7.9, U8.2
- new net GND4: C10.2, C9.2, J37.1, J42.3, J42.4, J43.1, J44.1, J45.1, U10.2, U9.14, U9.20, U9.25, U9.30, U9.34, U9.39, U9.6, U9.9
- new net GND5: C11.2, C12.2, J46.1, J51.3, J51.4, J52.1, J53.1, J54.1, U11.14, U11.20, U11.25, U11.30, U11.34, U11.39, U11.6, U11.9, U12.2
- new net GND6: C13.2, C14.2, J55.1, J60.3, J60.4, J61.1, J62.1, J63.1, U13.14, U13.20, U13.25, U13.30, U13.34, U13.39, U13.6, U13.9, U14.2
- new net GND7: C15.2, C16.2, J64.1, J69.3, J69.4, J70.1, J71.1, J72.1, U15.14, U15.20, U15.25, U15.30, U15.34, U15.39, U15.6, U15.9, U16.2
- new net ID_SCL1: U1.28
- new net ID_SCL2: U5.28
- new net ID_SCL3: U7.28
- new net ID_SCL4: U9.28
- new net ID_SCL5: U11.28
- new net ID_SCL6: U13.28
- new net ID_SCL7: U15.28
- new net ID_SDA1: U1.27
- new net ID_SDA2: U5.27
- new net ID_SDA3: U7.27
- new net ID_SDA4: U9.27
- new net ID_SDA5: U11.27
- new net ID_SDA6: U13.27
- new net ID_SDA7: U15.27
- new net MISO1: J14.2, U1.21
- new net MISO2: J23.2, U5.21
- new net MISO3: J32.2, U7.21
- new net MISO4: J41.2, U9.21
- new net MISO5: J50.2, U11.21
- new net MISO6: J59.2, U13.21
- new net MISO7: J68.2, U15.21
- new net MOSI1: J14.1, U1.19
- new net MOSI2: J23.1, U5.19
- new net MOSI3: J32.1, U7.19
- new net MOSI4: J41.1, U9.19
- new net MOSI5: J50.1, U11.19
- new net MOSI6: J59.1, U13.19
- new net MOSI7: J68.1, U15.19
- new net RX1: J13.2, U1.10
- new net RX2: J22.2, U5.10
- new net RX3: J31.2, U7.10
- new net RX4: J40.2, U9.10
- new net RX5: J49.2, U11.10
- new net RX6: J58.2, U13.10
- new net RX7: J67.2, U15.10
- new net SCK1: J14.3, U1.23
- new net SCK2: J23.3, U5.23
- new net SCK3: J32.3, U7.23
- new net SCK4: J41.3, U9.23
- new net SCK5: J50.3, U11.23
- new net SCK6: J59.3, U13.23
- new net SCK7: J68.3, U15.23
- new net SCL1: J11.2, J16.4, J17.4, J18.4, J9.4, U1.5
- new net SCL2: J19.4, J21.2, J25.4, J26.4, J27.4, U5.5
- new net SCL3: J28.4, J30.2, J34.4, J35.4, J36.4, U7.5
- new net SCL4: J37.4, J39.2, J43.4, J44.4, J45.4, U9.5
- new net SCL5: J46.4, J48.2, J52.4, J53.4, J54.4, U11.5
- new net SCL6: J55.4, J57.2, J61.4, J62.4, J63.4, U13.5
- new net SCL7: J64.4, J66.2, J70.4, J71.4, J72.4, U15.5
- new net SDA1: J11.1, J16.3, J17.3, J18.3, J9.3, U1.3
- new net SDA2: J19.3, J21.1, J25.3, J26.3, J27.3, U5.3
- new net SDA3: J28.3, J30.1, J34.3, J35.3, J36.3, U7.3
- new net SDA4: J37.3, J39.1, J43.3, J44.3, J45.3, U9.3
- new net SDA5: J46.3, J48.1, J52.3, J53.3, J54.3, U11.3
- new net SDA6: J55.3, J57.1, J61.3, J62.3, J63.3, U13.3
- new net SDA7: J64.3, J66.1, J70.3, J71.3, J72.3, U15.3
- new net TX1: J13.1, U1.8
- new net TX2: J22.1, U5.8
- new net TX3: J31.1, U7.8
- new net TX4: J40.1, U9.8
- new net TX5: J49.1, U11.8
- new net TX6: J58.1, U13.8
- new net TX7: J67.1, U15.8
Routing:
- net SDA5: track 0.00 -> 64.1 mm, vias 0 -> 3
- net SDA7: track 0.00 -> 64.1 mm, vias 0 -> 3
- net SDA4: track 0.00 -> 64.1 mm, vias 0 -> 3
- net SDA3: track 0.00 -> 64.1 mm, vias 0 -> 3
- net SDA2: track 0.00 -> 64.1 mm, vias 0 -> 3
- net SDA1: track 0.00 -> 64.1 mm, vias 0 -> 3
- net SDA6: track 0.00 -> 64.1 mm, vias 0 -> 3
- net SCL5: track 0.00 -> 55.7 mm
- net SCL4: track 0.00 -> 55.7 mm
- net SCL1: track 0.00 -> 55.7 mm
- net SCL7: track 0.00 -> 55.7 mm
- net SCL6: track 0.00 -> 55.7 mm
- net SCL3: track 0.00 -> 55.7 mm
- net SCL2: track 0.00 -> 55.7 mm
- net 3.3V7: track 0.00 -> 46.3 mm
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- added copper zone on layer 1, net GND1
- added copper zone on layer 16, net GND1
- added copper zone on layer 1, net GND2
- added copper zone on layer 16, net GND2
- added copper zone on layer 1, net GND3
- added copper zone on layer 16, net GND3
- added copper zone on layer 1, net GND4
- added copper zone on layer 16, net GND4
- added copper zone on layer 1, net GND5
- added copper zone on layer 16, net GND5
- added copper zone on layer 1, net GND6
- added copper zone on layer 16, net GND6
- added copper zone on layer 1, net GND7
- added copper zone on layer 16, net GND7
Other:
- board size 52.3 x 23 mm -> 126 x 100.3 mm
- board text added: "Mill Out"
- board text added: "Vscore"
- board text removed: "N. Seidle"
